Commit message: feat: implement clean RGB-D perception and refined documentation

File: src/fieldbot/urdf/fieldbot.urdf (robot description, URDF)
Before this commit: robot fieldbot, 6 links, 5 joints
Links:
- added link camera_link; visual box size=0.05 0.05 0.05
- added link camera_link_optical
Joints:
- added joint camera_joint: type fixed, parent base_link, child camera_link, origin xyz=0.55 0 0.3 rpy=0 0 0
- added joint camera_optical_joint: type fixed, parent camera_link, child camera_link_optical, origin xyz=0 0 0 rpy=-1.5707 0 -1.5707

Commit message: feat: Initial commit - GPS/IMU/EKF sensor fusion implementation
FieldBot autonomous agricultural navigation stack featuring:

- GPS/IMU/EKF dual-sensor fusion for outdoor localization
- RGB-D 3D perception with corrected optical frames
- Nav2 path planning and autonomous navigation
- Agricultural row surveyor tool for GPS waypoint recording
- Event-driven deterministic launch architecture
- Dual simulation environments (navigation + vineyard)

Tech stack:
- ROS 2 Jazzy Jalisco
- Gazebo Harmonic
- robot_localization (Dual-EKF)
- Nav2 with Regulated Pure Pursuit controller
- ros2_control for hardware abstraction

This implementation uses GPS-based absolute positioning suitable for
outdoor agricultural environments, NOT SLAM or AMCL.

File: src/fieldbot/urdf/fieldbot.urdf (robot description, URDF)
Before this commit: robot fieldbot, 8 links, 7 joints
Links:
- added link gps_link
- added link imu_link
Joints:
- added joint gps_joint: type fixed, parent base_link, child gps_link, origin xyz=0 0 0.4 rpy=0 0 0
- added joint imu_joint: type fixed, parent base_link, child imu_link, origin xyz=0 0 0.1 rpy=0 0 0
